File: pcb/_autosave-right.kicad_sch (KiCad schematic)
At the start: 47 parts, among them J1 OLED Connector, J2 Tag connect TC2030-CTX, J4 Conn_01x01_Socket, J5 Conn_01x01_Socket, SW1 RESET, SW23 EC11 Encoder, SW24 ON/OFF, U1 nRF52840, U4 DRV2605LDGS, Y1 32MHz, Y2 32.768kHz

Commit message: update everything
Parts:
- H1, H2, H3, H4, H5: footprint (none) -> MountingHole:MountingHole_2.2mm_M2
Other:
- moved on the sheet: H1
