File: pcb/keymatrix_right.kicad_sch (KiCad schematic)
At the start: 42 parts, among them SW10 SW_Push, SW11 SW_Push, SW12 SW_Push, SW13 SW_Push, SW14 SW_Push, SW15 SW_Push, SW16 SW_Push, SW17 SW_Push, SW18 SW_Push, SW19 SW_Push, SW2 SW_Push, SW20 SW_Push, SW21 SW_Push, SW22 SW_Push, SW3 SW_Push, SW4 SW_Push, SW5 SW_Push, SW6 SW_Push, SW7 SW_Push, SW8 SW_Push, SW9 SW_Push

Commit message: finished routing second half
Other:
- note added: "Kailh Hotswap Sockets can be assembled by PCBA. 42 * $0.04 = $1.68 cost for board extended part so there is a loading fee"
