File: pcb/pcb.kicad_sch (KiCad schematic)
At the start: 0 parts

Commit message: update everything
Other:
- note added: "both sides are identical except for GPIO pinouts"
Changed lines of the file:
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@@
 	(title_block
 		(title "k42 - Root File")
-		(date "2026-06-16")
+		(date "2026-06-24")
 		(rev "1.0.0")
 		(company "Dylan DiBeneditto")
 	)
+	(text "both sides are identical\nexcept for GPIO pinouts"
+		(exclude_from_sim no)
+		(at 151.13 163.322 0)
+		(effects
+			(font
+				(size 1.27 1.27)
+			)
+		)
+	)
 	(sheet
