File: pcb/power_left.kicad_sch (KiCad schematic)
At the start: 20 parts, among them J3 USB C 2.0 Connector, Q1 BSS84, Q2 BSS138, U2 BQ24073RGT, U3 USBLC6-2SC6

Commit message: update everything
Parts:
- removed BT1: Lipo Cell, Connector_JST:JST_PH_S2B-PH-SM4-TB_1x02-1MP_P2.00mm_Horizontal, symbol Device:Battery_Cell
- removed C20: 1u, Capacitor_SMD:C_0603_1608Metric, symbol Device:C_Small
- removed C22, C25: 4u7, Capacitor_SMD:C_0805_2012Metric, symbol Device:C_Small
- removed C26: 100n, Capacitor_SMD:C_0402_1005Metric, symbol Device:C_Small
- removed J3: USB C 2.0 Connector, kbd:TYPE-C-31-M-13C, symbol Connector:USB_C_Receptacle_USB2.0_16P
- removed Q1: BSS84, Package_TO_SOT_SMD:SOT-23, symbol Transistor_FET:BSS84
- removed Q2: BSS138, Package_TO_SOT_SMD:SOT-23, symbol Transistor_FET:BSS138
- removed R1: 100k, Resistor_SMD:R_0603_1608Metric, symbol Device:R_Small
- removed R2, R3: 5k1, Resistor_SMD:R_0402_1005Metric, symbol Device:R_Small
- removed R4, R6, R8, R9: 10k, Resistor_SMD:R_0402_1005Metric, symbol Device:R_Small
- removed R5: 3k2, Resistor_SMD:R_0402_1005Metric, symbol Device:R_Small
- removed R7: 5k9, Resistor_SMD:R_0402_1005Metric, symbol Device:R_Small
- removed TH1: 10k, Resistor_SMD:R_0402_1005Metric, symbol Device:Thermistor_NTC
- removed U2: BQ24073RGT, Package_DFN_QFN:VQFN-16-1EP_3x3mm_P0.5mm_EP1.6x1.6mm, symbol Battery_Management:BQ24073RGT
- removed U3: USBLC6-2SC6, Package_TO_SOT_SMD:SOT-23-6, symbol Power_Protection:USBLC6-2SC6
- added BT3: Lipo Cell, Connector_JST:JST_PH_S2B-PH-SM4-TB_1x02-1MP_P2.00mm_Horizontal, symbol Device:Battery_Cell
- added C53: 1u, Capacitor_SMD:C_0603_1608Metric, symbol Device:C_Small
- added C54, C55: 4u7, Capacitor_SMD:C_0805_2012Metric, symbol Device:C_Small
- added C56: 100n, Capacitor_SMD:C_0402_1005Metric, symbol Device:C_Small
- added J11: USB C 2.0 Connector, kbd:TYPE-C-31-M-13C, symbol Connector:USB_C_Receptacle_USB2.0_16P
- added Q5: BSS84, Package_TO_SOT_SMD:SOT-23, symbol Transistor_FET:BSS84
- added Q6: BSS138, Package_TO_SOT_SMD:SOT-23, symbol Transistor_FET:BSS138
- added R23: 100k, Resistor_SMD:R_0603_1608Metric, symbol Device:R_Small
- added R24, R25: 5k1, Resistor_SMD:R_0402_1005Metric, symbol Device:R_Small
- added R26, R28, R30, R31: 10k, Resistor_SMD:R_0402_1005Metric, symbol Device:R_Small
- added R27: 3k2, Resistor_SMD:R_0402_1005Metric, symbol Device:R_Small
- added R29: 5k9, Resistor_SMD:R_0402_1005Metric, symbol Device:R_Small
- added TH3: 10k, Resistor_SMD:R_0402_1005Metric, symbol Device:Thermistor_NTC
- added U10: USBLC6-2SC6, Package_TO_SOT_SMD:SOT-23-6, symbol Power_Protection:USBLC6-2SC6
- added U9: BQ24073RGT, Package_DFN_QFN:VQFN-16-1EP_3x3mm_P0.5mm_EP1.6x1.6mm, symbol Battery_Management:BQ24073RGT
Connections:
- net +BATT: now also BT3.1 (+), C55.1, Q5.3 (D), R23.1, U9.2 (BAT), U9.3 (BAT)
- net GND: now also BT3.2 (-), C53.2, C54.2, C55.2, C56.2, J11.A1 (GND), J11.A12 (GND), J11.B1 (GND), J11.B12 (GND), J11.S1 (SHIELD), Q6.2 (S), R24.2, R25.1, R27.1, R28.2, R29.1, TH3.2, U10.2 (GND), U9.15 (TD), U9.17 (VSS), U9.5 (EN2), U9.8 (VSS)
- net SENSE_EN: now also Q6.1 (G)
- net USB_CONN_D+: now also J11.A6 (D+), J11.B6 (D+), U10.3 (I/O2)
- net USB_CONN_D-: now also J11.A7 (D-), J11.B7 (D-), U10.1 (I/O1)
- net USB_D+: now also U10.4 (I/O2)
- net USB_D-: now also U10.6 (I/O1)
- net VBAT_SENSE: now also C56.1, R26.2, R28.1
- net VBUS: now also C53.1, J11.A4 (VBUS), J11.A9 (VBUS), J11.B4 (VBUS), J11.B9 (VBUS), U10.5 (VBUS), U9.13 (IN), U9.6 (EN1)
- net V_{SYS}: now also C54.1, U9.10 (OUT), U9.11 (OUT)
- net ~{CHG}: now also R31.2
- net ~{PGOOD}: now also R30.2
- new net: J11.A5 (CC1), R24.1
- new net: J11.B5 (CC2), R25.2
- new net: Q5.1 (G), Q6.3 (D), R23.2
- new net: Q5.2 (S), R26.1
- new net: R30.1, U9.7 (~{PGOOD})
- new net: TH3.1, U9.1 (TS)
- new net: R27.2, U9.12 (ILIM)
- new net: R29.2, U9.16 (ISET)
- new net: R31.1, U9.9 (~{CHG})
- new net ~{CE}: U9.4 (~{CE})
Other:
- note removed: "(ran out of pins)"
- title: Right Half Power -> (none)

Commit message: finished routing second half
Connections:
- net GND: now also U9.4 (~{CE})
- net ~{CE}: no longer U9.4 (~{CE})
