File: pcb/power_right.kicad_sch (KiCad schematic)
At the start: 20 parts, among them J3 USB C 2.0 Connector, Q1 BSS84, Q2 BSS138, U2 BQ24073RGT, U3 USBLC6-2SC6

Commit message: finished routing second half
Parts:
- BT1: price (none) -> 1.20
- J3: price (none) -> 0.07
- U2: price (none) -> 0.88
- U3: price (none) -> 0.18
