File: pcb/right.kicad_sch (KiCad schematic)
At the start: 47 parts, among them J1 OLED Connector, J2 Tag connect TC2030-CTX, J4 Conn_01x01_Socket, J5 Conn_01x01_Socket, SW1 RESET, SW23 EC11 Encoder, SW24 ON/OFF, U1 nRF52840, U4 DRV2605LDGS, Y1 32MHz, Y2 32.768kHz

Commit message: finished routing second half
Parts:
- H1, H2, H3, H4, H5: footprint (none) -> MountingHole:MountingHole_2.2mm_M2
- J1, SW23: price (none) -> 0.90
- J4, J5: price (none) -> 0.03
- SW1: price (none) -> 0.05
- SW24: price (none) -> 0.07
- U1: price (none) -> 6.00
- U4: price (none) -> 1.18
- Y1: price (none) -> 0.12
- Y2: price (none) -> 0.17
Connections:
- net ROW 0: now also U1.B19 (P1.11); no longer U1.J24 (NFC2/P0.10)
- net ~{CHG}: now also U1.J24 (NFC2/P0.10); no longer U1.B19 (P1.11)

Commit message: impedence matched 50ohms and adjusted pi network
Parts:
- removed L9: 2.2nH, Inductor_SMD:L_0402_1005Metric, symbol Device:L_Small
- C18: value 1.2p -> 0.5pF
- C19: value 1p -> 0.8pF
Connections:
- net at AE1.1 (A), C23.1: now also C18.1, L5.1
Changed lines of the file:
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@@
 	(wire
 		(pts
-			(xy 31.75 73.66) (xy 34.29 73.66)
-		)
-		(stroke
-			(width 0)
-			(type default)
-		)
-	)
-	(wire
-		(pts
 			(xy 142.24 59.69) (xy 142.24 58.42)
 		)
@@
 	(wire
 		(pts
-			(xy 24.13 73.66) (xy 26.67 73.66)
+			(xy 24.13 73.66) (xy 34.29 73.66)
 		)
 		(stroke
@@
 			)
 		)
-		(property "Value" "1.2p"
+		(property "Value" "0.5pF"
 			(at 36.83 80.0162 0)
 			(show_name no)
@@
 	)
 	(symbol
-		(lib_id "Device:L_Small")
-		(at 29.21 73.66 90)
-		(unit 1)
-		(body_style 1)
-		(exclude_from_sim no)
-		(in_bom yes)
-		(on_board yes)
-		(in_pos_files yes)
-		(dnp no)
-		(fields_autoplaced yes)
-		(property "Reference" "L9"
-			(at 29.21 68.58 90)
-			(show_name no)
-			(do_not_autoplace no)
-			(effects
-				(font
-					(size 1.27 1.27)
-				)
-			)
-		)
-		(property "Value" "2.2nH"
-			(at 29.21 71.12 90)
-			(show_name no)
-			(do_not_autoplace no)
-			(effects
-				(font
-					(size 1.27 1.27)
-				)
-			)
-		)
-		(property "Footprint" "Inductor_SMD:L_0402_1005Metric"
-			(at 29.21 73.66 0)
-			(hide yes)
-			(show_name no)
-			(do_not_autoplace no)
-			(effects
-				(font
-					(size 1.27 1.27)
-				)
-			)
-		)
-		(property "Datasheet" ""
-			(at 29.21 73.66 0)
-			(hide yes)
-			(show_name no)
-			(do_not_autoplace no)
-			(effects
-				(font
-					(size 1.27 1.27)
-				)
-			)
-		)
-		(property "Description" "Inductor, small symbol"
-			(at 29.21 73.66 0)
-			(hide yes)
-			(show_name no)
-			(do_not_autoplace no)
-			(effects
-				(font
-					(size 1.27 1.27)
-				)
-			)
-		)
-		(pin "1"
-		)
-		(pin "2"
-		)
-		(instances
-			(project "pcb"
-				(path "/79b359b8-94d1-439d-a17f-41f5d59081a6/b2c8f017-14f5-4783-8c1b-fe907bb97694"
-					(reference "L9")
-					(unit 1)
-				)
-			)
-		)
-	)
-	(symbol
 		(lib_id "power:GND")
 		(at 19.05 83.82 0)
@@
 			)
 		)
-		(property "Value" "1p"
+		(property "Value" "0.8pF"
 			(at 46.99 80.0162 0)
 			(show_name no)
