File: pcb/pcb.kicad_pcb (KiCad board)
At the start: 2 copper layers, 10.5 x 10.5 mm, 96 parts, among them J1 Conn_Haptic_LRA, J2 Conn_01x02_Pin, SW1 SW_Push, SW10 SW_Push, SW11 SW_Push, SW12 SW_Push, SW13 SW_Push, SW14 SW_Push, SW15 SW_Push, SW16 SW_Push, SW17 SW_Push, SW18 SW_Push, SW19 SW_Push, SW2 SW_Push, SW20 SW_Push, SW21 SW_Push, SW22 RotaryEncoder_Switch_MP, SW23 SW_SPDT, SW24 SW_Reset, SW3 SW_Push, SW4 SW_Push, SW5 SW_Push, SW6 SW_Push, SW7 SW_Push, SW8 SW_Push, SW9 SW_Push, U1 DRV2605LDGS

Commit message: matrix wiring complete
Parts:
- removed the H1 at (154.3, 110.6)
- removed the H2 at (128.8, 48.7)
- removed the H4 at (52.8, 48.7)
- removed the H5 at (52.8, 84.7)
- removed SW24: SW_Reset, Capacitor_THT:CP_Axial_L10.0mm_D4.5mm_P15.00mm_Horizontal
- added D1: 1N4148W, Diode_SMD:D_SOD-123, B.Cu at (78.5, 58.7)
- added D10: 1N4148W, Diode_SMD:D_SOD-123, B.Cu at (135.5, 74.4)
- added D11: 1N4148W, Diode_SMD:D_SOD-123, B.Cu at (154.7, 77.4)
- added D12: 1N4148W, Diode_SMD:D_SOD-123, B.Cu at (173.7, 77.4)
- added D13: 1N4148W, Diode_SMD:D_SOD-123, B.Cu at (78.3, 96.4)
- added D14: 1N4148W, Diode_SMD:D_SOD-123, B.Cu at (97.4, 96.4)
- added D15: 1N4148W, Diode_SMD:D_SOD-123, B.Cu at (116.5, 94.2)
- added D16: 1N4148W, Diode_SMD:D_SOD-123, B.Cu at (135.5, 93.4)
- added D17: 1N4148W, Diode_SMD:D_SOD-123, B.Cu at (154.5, 96.4)
- added D18: 1N4148W, Diode_SMD:D_SOD-123, B.Cu at (173.7, 96.7)
- added D19: 1N4148W, Diode_SMD:D_SOD-123, B.Cu at (154.6, 117.7)
- added D2: 1N4148W, Diode_SMD:D_SOD-123, B.Cu at (97.2, 58.7)
- added D20: 1N4148W, Diode_SMD:D_SOD-123, B.Cu at (179.2, 119.4)
- added D21: 1N4148W, Diode_SMD:D_SOD-123, B.Cu at (200.8, 127.7)
- added D3: 1N4148W, Diode_SMD:D_SOD-123, B.Cu at (116.5, 55.9)
- added D4: 1N4148W, Diode_SMD:D_SOD-123, B.Cu at (135.7, 55.4)
- added D5: 1N4148W, Diode_SMD:D_SOD-123, B.Cu at (154.5, 58.4)
- added D6: 1N4148W, Diode_SMD:D_SOD-123, B.Cu at (173.5, 58.4)
- added D7: 1N4148W, Diode_SMD:D_SOD-123, B.Cu at (78.2, 77.7)
- added D8: 1N4148W, Diode_SMD:D_SOD-123, B.Cu at (97.5, 77.7)
- added D9: 1N4148W, Diode_SMD:D_SOD-123, B.Cu at (116.5, 74.9)
- added H6: MountingHole, MountingHole:MountingHole_2.2mm_M2, F.Cu at (93.9, 123.0)
- added REF**: LRA hole, kbd:LRA hole, F.Cu at (187.8, 97.9)
- added REF**: Breakaway_Tabs, kbd:Breakaway_Tabs, F.Cu at (101.2, 117.0)
- added SW23: SW_SPDT, Button_Switch_SMD:SW_SPDT_PCM12, B.Cu at (189.2, 57.5)
- added U1: DRV2605LDGS, Package_SO:TSSOP-10_3x3mm_P0.5mm, B.Cu at (203.8, 104.8)
- JP1: moved to F.Cu
- JP10, JP12, JP2: moved to B.Cu
- moved D13 170.1 mm to (78.3, 96.4), turned to 180 degrees
- moved D7 162.3 mm to (78.2, 77.7), turned to 180 degrees
- moved D1 162.1 mm to (78.5, 58.7), turned to 180 degrees
- moved D14 150.7 mm to (97.4, 96.4), turned to 180 degrees
- moved D2 143.4 mm to (97.2, 58.7), turned to 180 degrees
- moved D8 143.1 mm to (97.5, 77.7), turned to 180 degrees
- moved D9 131.2 mm to (116.5, 74.9), turned to 180 degrees
- moved D15 131.0 mm to (116.5, 94.2), turned to 180 degrees
- moved D3 124.3 mm to (116.5, 55.9), turned to 180 degrees
- moved D10 111.8 mm to (135.5, 74.4), turned to 180 degrees
- moved D16 111.7 mm to (135.5, 93.4), turned to 180 degrees
- moved D19 111.6 mm to (154.6, 117.7), turned to 180 degrees
- moved D4 105.5 mm to (135.7, 55.4), turned to 180 degrees
- moved D17 105.4 mm to (154.5, 96.4), turned to 180 degrees
- moved D11 92.7 mm to (154.7, 77.4), turned to 180 degrees
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Connections:
- JP1 pad 1: GND -> SDA
- JP12 pad 2: Net-(J2-Pin_2) -> Net-(J2-Pin_1)
- JP3 pad 1: +3V3 -> SCL
- JP5 pad 1: SCL -> +3V3
- JP7 pad 1: SDA -> GND
- JP9 pad 1: Net-(J2-Pin_1) -> Net-(J2-Pin_2)
- U1 pad 7: Net-(J1-Pin_1) -> Net-(J1-Pin_2)
- U1 pad 9: Net-(J1-Pin_2) -> Net-(J1-Pin_1)
- U3 pad 1: VBAT_SW -> (no net)
- U3 pad 11: BOTTOM -> (no net)
- U3 pad 12: THUMB -> (no net)
- U3 pad 13: CENTER -> (no net)
- U3 pad 14: TOP -> (no net)
- U3 pad 15: INNER -> (no net)
- U3 pad 16: INDEX -> (no net)
- U3 pad 17: MIDDLE -> (no net)
- U3 pad 18: RING -> (no net)
- U3 pad 19: PINKY -> (no net)
- U3 pad 2: GND -> (no net)
- U3 pad 20: OUTER -> (no net)
- U3 pad 21: GND -> (no net)
- U3 pad 22: GND -> (no net)
- U3 pad 23: SCL -> (no net)
- U3 pad 24: SDA -> (no net)
- U3 pad 3: RST -> (no net)
- U3 pad 4: +3V3 -> (no net)
- U3 pad 5: HAPTIC_EN -> (no net)
- U3 pad 6: EC_A -> (no net)
- U3 pad 7: EC_B -> (no net)
- U3 pad 8: EC_SW -> (no net)
Routing:
- net INNER: track 0.00 -> 175.4 mm, vias 0 -> 4
- net MIDDLE: track 0.00 -> 170.9 mm, vias 0 -> 4
- net INDEX: track 0.00 -> 170.0 mm, vias 0 -> 4
- net CENTER: track 0.00 -> 125.2 mm, vias 0 -> 6
- net TOP: track 0.00 -> 125.1 mm, vias 0 -> 6
- net BOTTOM: track 0.00 -> 124.1 mm, vias 0 -> 6
- net RING: track 0.00 -> 112.5 mm, vias 0 -> 3
- net PINKY: track 0.00 -> 111.5 mm, vias 0 -> 3
- net OUTER: track 0.00 -> 111.5 mm, vias 0 -> 3
- net THUMB: track 0.00 -> 56.9 mm, vias 0 -> 3
- net VBAT_SW: track 0.00 -> 27.0 mm, vias 0 -> 1
- net Net-(D20-A): track 0.00 -> 24.0 mm, vias 0 -> 1
- net Net-(D14-A): track 0.00 -> 23.5 mm, vias 0 -> 1
- net Net-(D2-A): track 0.00 -> 23.5 mm, vias 0 -> 1
- net Net-(D13-A): track 0.00 -> 23.4 mm, vias 0 -> 1
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- added copper zone on B.Cu, net GND
- added copper zone on F.Cu, net GND
Other:
- board size 10.5 x 10.5 mm -> 145.2 x 98.5 mm
- board text added: "bridge if TOP"
- board text added: "bridge to RST"
- board text removed: "if this is the bottom solder all jumpers together"

Commit message: finished routing
Connections:
- U3 pad 1: (no net) -> VBAT_SW
- U3 pad 11: (no net) -> OUTER
- U3 pad 12: (no net) -> THUMB
- U3 pad 13: (no net) -> PINKY
- U3 pad 14: (no net) -> RING
- U3 pad 15: (no net) -> MIDDLE
- U3 pad 16: (no net) -> INDEX
- U3 pad 17: (no net) -> INNER
- U3 pad 18: (no net) -> BOTTOM
- U3 pad 19: (no net) -> CENTER
- U3 pad 2: (no net) -> GND
- U3 pad 20: (no net) -> TOP
- U3 pad 21: (no net) -> GND
- U3 pad 22: (no net) -> GND
- U3 pad 23: (no net) -> SCL
- U3 pad 24: (no net) -> SDA
- U3 pad 3: (no net) -> RST
- U3 pad 4: (no net) -> +3V3
- U3 pad 5: (no net) -> HAPTIC_EN
- U3 pad 6: (no net) -> EC_A
- U3 pad 7: (no net) -> EC_B
- U3 pad 8: (no net) -> EC_SW
Routing:
- net OUTER: track 111.5 -> 259.8 mm
- net PINKY: track 111.5 -> 225.3 mm
- net RING: track 112.5 -> 211.5 mm
- net MIDDLE: track 170.9 -> 254.0 mm
- net +3V3: track 0.00 -> 68.2 mm, vias 0 -> 4
- net INDEX: track 170.0 -> 233.7 mm
- net SDA: track 0.00 -> 62.7 mm, vias 0 -> 3
- net EC_B: track 0.00 -> 61.7 mm, vias 0 -> 3
- net SCL: track 0.00 -> 61.6 mm, vias 0 -> 3
- net EC_SW: track 0.00 -> 58.3 mm, vias 0 -> 3
- net EC_A: track 0.00 -> 50.6 mm, vias 0 -> 3
- net HAPTIC_EN: track 0.00 -> 46.4 mm, vias 0 -> 1
- net THUMB: track 56.9 -> 100.2 mm
- net BOTTOM: track 124.1 -> 157.7 mm
- net TOP: track 125.1 -> 152.0 mm
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
Commit message: finishing touches to routing
Routing:
- net SCL: track 61.6 -> 63.2 mm
- net GND: vias 41 -> 26
Other:
- board text removed: "bridge if TOP"

Commit message: update
Routing:
- net GND: vias 26 -> 22
Other:
- board text added: "Don't overtighten"
- board text added: "LRA Here"
- board text removed: "bridge to RST"
