File: pcb/_restore_backup_2026-07-24T13-59-45-257/pcb.kicad_sch (KiCad schematic)
At the start: 72 parts, among them J1 Conn_Haptic_LRA, J2 Conn_01x02_Pin, SW1 SW_Push, SW10 SW_Push, SW11 SW_Push, SW12 SW_Push, SW13 SW_Push, SW14 SW_Push, SW15 SW_Push, SW16 SW_Push, SW17 SW_Push, SW18 SW_Push, SW19 SW_Push, SW2 SW_Push, SW20 SW_Push, SW21 SW_Push, SW22 RotaryEncoder_Switch_MP, SW23 SW_SPDT, SW24 SW_Reset, SW3 SW_Push, SW4 SW_Push, SW5 SW_Push, SW6 SW_Push, SW7 SW_Push, SW8 SW_Push, SW9 SW_Push, U1 DRV2605LDGS

Commit message: matrix wiring complete
Connections:
- net +3V3: now also JP3.1 (A); no longer JP5.1 (A)
- net GND: now also JP1.1 (A); no longer JP7.1 (A)
- net SCL: now also JP5.1 (A); no longer JP3.1 (A)
- net SDA: now also JP7.1 (A); no longer JP1.1 (A)
- net at J2.1 (Pin_1), JP10.2 (B): now also JP9.1 (A); no longer JP12.2 (B)
- net at J1.1 (Pin_1): now also U1.7 (OUT+); no longer U1.9 (OUT-)
- net at J1.2 (Pin_2): now also U1.9 (OUT-); no longer U1.7 (OUT+)
- net at J2.2 (Pin_2), JP11.1 (A): now also JP12.2 (B); no longer JP9.1 (A)
